Commit message: base link is now visible and has inertial component

File: phoebe.urdf (robot description, URDF)
Before this commit: robot phoebe, 38 links, 37 joints
Links:
- removed link bumblebee_cameras_link
- removed link bumblebee_link
- removed link hokuyo_link
- removed link left_arm_base_link
- removed link left_arm_camera
- removed link left_arm_camera_bracket
- removed link left_arm_elbow_pitch
- removed link left_arm_elbow_yaw
- removed link left_arm_gripper_finger1
- removed link left_arm_gripper_finger2
- removed link left_arm_shoulder_pitch
- removed link left_arm_shoulder_roll
- removed link left_arm_shoulder_yaw
- removed link left_arm_virtual_endeffector
- removed link left_arm_wrist_pitch
- removed link left_arm_wrist_roll
- removed link ptu_base_link
- removed link ptu_base_plate_link
- removed link ptu_mount_link
- removed link ptu_pan_link
- removed link ptu_tilt_link
- removed link right_arm_base_link
- removed link right_arm_camera
- removed link right_arm_camera_bracket
- removed link right_arm_elbow_pitch
- removed link right_arm_elbow_yaw
- removed link right_arm_gripper_finger1
- removed link right_arm_gripper_finger2
- removed link right_arm_shoulder_pitch
- removed link right_arm_shoulder_roll
- removed link right_arm_shoulder_yaw
- removed link right_arm_virtual_endeffector
- removed link right_arm_wrist_pitch
- removed link right_arm_wrist_roll
- removed link wheel_left
- removed link wheel_right
- removed link xtion_link
- link base_link: mass None -> 12
Joints:
- removed joint bumblebee_cameras_joint
- removed joint bumblebee_joint
- removed joint hokuyo_base_joint
- removed joint left_arm_camera_bracket_joint
- removed joint left_arm_camera_joint
- removed joint left_arm_elbow_pitch_joint
- removed joint left_arm_elbow_yaw_joint
- removed joint left_arm_gripper_joint
- removed joint left_arm_gripper_joint2
- removed joint left_arm_joint
- removed joint left_arm_shoulder_pitch_joint
- removed joint left_arm_shoulder_roll_joint
- removed joint left_arm_shoulder_yaw_joint
- removed joint left_arm_virtual_endeffector_joint
- removed joint left_arm_wrist_pitch_joint
- removed joint left_arm_wrist_roll_joint
- removed joint ptu_base_joint
- removed joint ptu_base_plate_joint
- removed joint ptu_joint
- removed joint ptu_pan_joint
- removed joint ptu_tilt_joint
- removed joint right_arm_camera_bracket_joint
- removed joint right_arm_camera_joint
- removed joint right_arm_elbow_pitch_joint
- removed joint right_arm_elbow_yaw_joint
- removed joint right_arm_gripper_joint
- removed joint right_arm_gripper_joint2
- removed joint right_arm_joint
- removed joint right_arm_shoulder_pitch_joint
- removed joint right_arm_shoulder_roll_joint
- removed joint right_arm_shoulder_yaw_joint
- removed joint right_arm_virtual_endeffector_joint
- removed joint right_arm_wrist_pitch_joint
- removed joint right_arm_wrist_roll_joint
- removed joint wheel_left_joint
- removed joint wheel_right_joint
- removed joint xtion_joint

Commit message: added inertial parameters for links

File: phoebe.urdf (robot description, URDF)
Before this commit: robot phoebe, 1 links, 0 joints
Links:
- added link bumblebee_cameras_link; visual cylinder length=0.001 radius=0.011; visual cylinder length=0.001 radius=0.011
- added link bumblebee_link, mass 0.342; visual box size=0.047 0.157 0.038
- added link hokuyo_link, mass 0.13; collision box size=0.05 0.05 0.041; collision cylinder length=0.0265 radius=0.021
- added link left_arm_base_link, mass 0.478571; collision box size=0.154 0.177 0.094; visual mesh filename=package://cyton_gamma_1500_description/meshes/base.dae
- added link left_arm_camera, mass 0.085; collision box size=0.036 0.045 0.063; visual box size=0.031 0.028 0.063
- added link left_arm_camera_bracket, mass 0.052; visual mesh filename=package://cyton_gamma_1500_minicam_description/meshes/cam_b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
- added link left_arm_elbow_pitch, mass 0.388671; collision box size=0.0549 0.1557 0.076; visual mesh filename=package://cyton_gamma_1500_description/meshes/elbow_pitch.d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
- added link left_arm_elbow_yaw, mass 0.368871; collision box size=0.0535 0.1160 0.0402; visual mesh filename=package://cyton_gamma_1500_description/meshes/elbow_yaw.dae
- added link left_arm_gripper_finger1, mass 0.035; collision box size=0.015 0.0229 0.0475; visual mesh filename=package://cyton_gamma_1500_description/meshes/gripper_finge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
- added link left_arm_gripper_finger2, mass 0.035; collision box size=0.015 0.0229 0.0475; visual mesh filename=package://cyton_gamma_1500_description/meshes/gripper_finge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
- added link left_arm_shoulder_pitch, mass 0.4285714; collision box size=0.0709 0.19363 0.083; visual mesh filename=package://cyton_gamma_1500_description/meshes/shoulder_pitc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
- added link left_arm_shoulder_roll, mass 0.468571; collision box size=0.09829 0.18143 0.08392; visual mesh filename=package://cyton_gamma_1500_description/meshes/shoulder_roll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
- added link left_arm_shoulder_yaw, mass 0.408571; collision box size=0.0717 0.1846 0.0756; visual mesh filename=package://cyton_gamma_1500_description/meshes/shoulder_yaw.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
- added link left_arm_virtual_endeffector, mass 0.0016; visual sphere radius=0.002
- added link left_arm_wrist_pitch, mass 0.008; collision box size=0.026 0.0435 0.05185; visual mesh filename=package://cyton_gamma_1500_description/meshes/wrist_pitch.d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
- added link left_arm_wrist_roll, mass 0.38; collision box size=0.0518 0.0723 0.1004; visual mesh filename=package://cyton_gamma_1500_description/meshes/wrist_roll.dae
- added link ptu_base_link
- added link ptu_base_plate_link, mass 0.07; visual box size=0.17 0.142 0.005
- added link ptu_mount_link, mass 0.07; collision box size=0.154 0.177 0.094; visual mesh filename=package://dp_ptu_46_description/meshes/mount.dae
- added link ptu_pan_link, mass 0.13; collision box size=0.154 0.177 0.094; visual mesh filename=package://dp_ptu_46_description/meshes/pan.dae
- added link ptu_tilt_link, mass 0.13; collision box size=0.154 0.177 0.094; visual mesh filename=package://dp_ptu_46_description/meshes/tilt.dae
- added link right_arm_base_link, mass 0.478571; collision box size=0.154 0.177 0.094; visual mesh filename=package://cyton_gamma_1500_description/meshes/base.dae
- added link right_arm_camera, mass 0.085; collision box size=0.036 0.045 0.063; visual box size=0.031 0.028 0.063
- added link right_arm_camera_bracket, mass 0.052; visual mesh filename=package://cyton_gamma_1500_minicam_description/meshes/cam_b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
- added link right_arm_elbow_pitch, mass 0.388671; collision box size=0.0549 0.1557 0.076; visual mesh filename=package://cyton_gamma_1500_description/meshes/elbow_pitch.d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
- added link right_arm_elbow_yaw, mass 0.368871; collision box size=0.0535 0.1160 0.0402; visual mesh filename=package://cyton_gamma_1500_description/meshes/elbow_yaw.dae
- added link right_arm_gripper_finger1, mass 0.035; collision box size=0.015 0.0229 0.0475; visual mesh filename=package://cyton_gamma_1500_description/meshes/gripper_finge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
- added link right_arm_gripper_finger2, mass 0.035; collision box size=0.015 0.0229 0.0475; visual mesh filename=package://cyton_gamma_1500_description/meshes/gripper_finge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
- added link right_arm_shoulder_pitch, mass 0.4285714; collision box size=0.0709 0.19363 0.083; visual mesh filename=package://cyton_gamma_1500_description/meshes/shoulder_pitc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
- added link right_arm_shoulder_roll, mass 0.468571; collision box size=0.09829 0.18143 0.08392; visual mesh filename=package://cyton_gamma_1500_description/meshes/shoulder_roll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
- added link right_arm_shoulder_yaw, mass 0.408571; collision box size=0.0717 0.1846 0.0756; visual mesh filename=package://cyton_gamma_1500_description/meshes/shoulder_yaw.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
- added link right_arm_virtual_endeffector, mass 0.0016; visual sphere radius=0.002
- added link right_arm_wrist_pitch, mass 0.008; collision box size=0.026 0.0435 0.05185; visual mesh filename=package://cyton_gamma_1500_description/meshes/wrist_pitch.d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
- added link right_arm_wrist_roll, mass 0.38; collision box size=0.0518 0.0723 0.1004; visual mesh filename=package://cyton_gamma_1500_description/meshes/wrist_roll.dae
- added link wheel_left, mass 0.5; collision cylinder length=0.05 radius=0.095; visual cylinder length=0.05 radius=0.095
- added link wheel_right, mass 0.5; collision cylinder length=0.05 radius=0.095; visual cylinder length=0.05 radius=0.095
- added link xtion_link, mass 0.54; visual box size=0.02 0.017 0.02; visual box size=0.036 0.178 0.03
Joints:
- added joint bumblebee_cameras_joint: type fixed, parent bumblebee_link, child bumblebee_cameras_link, origin xyz=0 0 0.0 rpy=0 0 0
- added joint bumblebee_joint: type fixed, parent ptu_mount_link, child bumblebee_link, origin xyz=0 0 0.058 rpy=0 0 0
- added joint hokuyo_base_joint: type fixed, parent base_link, child hokuyo_link, origin xyz=0.1 0 0.3 rpy=0 0 0
- added joint left_arm_camera_bracket_joint: type fixed, parent left_arm_wrist_roll, child left_arm_camera_bracket, origin xyz=-0.0008 -0.028 0.0435 rpy=0 0 0
- added joint left_arm_camera_joint: type fixed, parent left_arm_camera_bracket, child left_arm_camera, origin xyz=0.0 -0.028 -0.005 rpy=-0.625 0 0
- added joint left_arm_elbow_pitch_joint: type revolute, parent left_arm_shoulder_yaw, child left_arm_elbow_pitch, origin xyz=0.018 0.0206 0.1158 rpy=0 0 0, axis 1 0 0, limit lower=-1.8326 upper=1.8326 effort=100.0 velocity=1.0
- added joint left_arm_elbow_yaw_joint: type revolute, parent left_arm_elbow_pitch, child left_arm_elbow_yaw, origin xyz=-0.0171 -0.018 0.09746 rpy=0 0 0, axis 0 -1 0, limit lower=-1.8326 upper=1.8326 effort=100.0 velocity=1.0
- added joint left_arm_gripper_joint: type prismatic, parent left_arm_wrist_roll, child left_arm_gripper_finger1, origin xyz=-0.01331 0.00485 0.077225 rpy=0 0 0, axis 1 0 0, limit lower=-0.008 upper=0.008 effort=100.0 velocity=1.0
- added joint left_arm_gripper_joint2: type prismatic, parent left_arm_wrist_roll, child left_arm_gripper_finger2, origin xyz=0.0098 0.00485 0.077225 rpy=0 0 0, axis 1 0 0, limit lower=-0.008 upper=0.008 effort=100.0 velocity=1.0, mimic joint=left_arm_gripper_joint multiplier=-1
- added joint left_arm_joint: type fixed, parent base_link, child left_arm_base_link, origin xyz=0.067 0.162 0.8 rpy=-1.5708 1.5708 0
- added joint left_arm_shoulder_pitch_joint: type revolute, parent left_arm_shoulder_roll, child left_arm_shoulder_pitch, origin xyz=0.0205 0 0.12435 rpy=0 0 0, axis 1 0 0, limit lower=-1.8326 upper=1.8326 effort=100.0 velocity=1.0
- added joint left_arm_shoulder_roll_joint: type revolute, parent left_arm_base_link, child left_arm_shoulder_roll, origin xyz=0 0 0.05315 rpy=0 0 0, axis 0 0 1, limit lower=-2.618 upper=2.618 effort=100.0 velocity=1.0
- added joint left_arm_shoulder_yaw_joint: type revolute, parent left_arm_shoulder_pitch, child left_arm_shoulder_yaw, origin xyz=-0.0215 -0.0205 0.1255 rpy=0 0 0, axis 0 -1 0, limit lower=-1.8326 upper=1.8326 effort=100.0 velocity=1.0
- added joint left_arm_virtual_endeffector_joint: type fixed, parent left_arm_wrist_roll, child left_arm_virtual_endeffector, origin xyz=-0.002316 0.0079 0.079425 rpy=0 0 0
- added joint left_arm_wrist_pitch_joint: type revolute, parent left_arm_elbow_yaw, child left_arm_wrist_pitch, origin xyz=0.02626 0.018 0.0718 rpy=0 0 0, axis -1 0 0, limit lower=-1.8326 upper=1.8326 effort=100.0 velocity=1.0
- added joint left_arm_wrist_roll_joint: type revolute, parent left_arm_wrist_pitch, child left_arm_wrist_roll, origin xyz=-0.026255 0 0.051425 rpy=0 0 0, axis 0 0 1, limit lower=-2.61799 upper=2.61799 effort=100.0 velocity=1.0
- added joint ptu_base_joint: type fixed, parent ptu_base_link, child ptu_pan_link, origin xyz=0.0 0 0.005 rpy=0 0 0
- added joint ptu_base_plate_joint: type fixed, parent ptu_base_plate_link, child ptu_base_link, origin xyz=0.0 0.0 0.0 rpy=0 0 0
- added joint ptu_joint: type fixed, parent base_link, child ptu_base_plate_link, origin xyz=0.02 0 1.1075 rpy=0 0 0
- added joint ptu_pan_joint: type revolute, parent ptu_base_link, child ptu_tilt_link, origin xyz=-0.00436 -0.0067 0.03 rpy=0 0 0, axis 0 0 1, limit lower=-2.775 upper=2.775 effort=100.0 velocity=1.0
- added joint ptu_tilt_joint: type revolute, parent ptu_tilt_link, child ptu_mount_link, origin xyz=0.0 0 0.0659 rpy=0 0 0, axis 0 -1 0, limit lower=-1.396 upper=0.541 effort=100.0 velocity=1.0
- added joint right_arm_camera_bracket_joint: type fixed, parent right_arm_wrist_roll, child right_arm_camera_bracket, origin xyz=-0.0008 -0.028 0.0435 rpy=0 0 0
- added joint right_arm_camera_joint: type fixed, parent right_arm_camera_bracket, child right_arm_camera, origin xyz=0.0 -0.028 -0.005 rpy=-0.625 0 0
- added joint right_arm_elbow_pitch_joint: type revolute, parent right_arm_shoulder_yaw, child right_arm_elbow_pitch, origin xyz=0.018 0.0206 0.1158 rpy=0 0 0, axis 1 0 0, limit lower=-1.8326 upper=1.8326 effort=100.0 velocity=1.0
- added joint right_arm_elbow_yaw_joint: type revolute, parent right_arm_elbow_pitch, child right_arm_elbow_yaw, origin xyz=-0.0171 -0.018 0.09746 rpy=0 0 0, axis 0 -1 0, limit lower=-1.8326 upper=1.8326 effort=100.0 velocity=1.0
- added joint right_arm_gripper_joint: type prismatic, parent right_arm_wrist_roll, child right_arm_gripper_finger1, origin xyz=-0.01331 0.00485 0.077225 rpy=0 0 0, axis 1 0 0, limit lower=-0.008 upper=0.008 effort=100.0 velocity=1.0
- added joint right_arm_gripper_joint2: type prismatic, parent right_arm_wrist_roll, child right_arm_gripper_finger2, origin xyz=0.0098 0.00485 0.077225 rpy=0 0 0, axis 1 0 0, limit lower=-0.008 upper=0.008 effort=100.0 velocity=1.0, mimic joint=right_arm_gripper_joint multiplier=-1
- added joint right_arm_joint: type fixed, parent base_link, child right_arm_base_link, origin xyz=0.067 -0.162 0.8 rpy=1.5708 -1.5708 0
- added joint right_arm_shoulder_pitch_joint: type revolute, parent right_arm_shoulder_roll, child right_arm_shoulder_pitch, origin xyz=0.0205 0 0.12435 rpy=0 0 0, axis 1 0 0, limit lower=-1.8326 upper=1.8326 effort=100.0 velocity=1.0
- added joint right_arm_shoulder_roll_joint: type revolute, parent right_arm_base_link, child right_arm_shoulder_roll, origin xyz=0 0 0.05315 rpy=0 0 0, axis 0 0 1, limit lower=-2.618 upper=2.618 effort=100.0 velocity=1.0
- added joint right_arm_shoulder_yaw_joint: type revolute, parent right_arm_shoulder_pitch, child right_arm_shoulder_yaw, origin xyz=-0.0215 -0.0205 0.1255 rpy=0 0 0, axis 0 -1 0, limit lower=-1.8326 upper=1.8326 effort=100.0 velocity=1.0
- added joint right_arm_virtual_endeffector_joint: type fixed, parent right_arm_wrist_roll, child right_arm_virtual_endeffector, origin xyz=-0.002316 0.0079 0.079425 rpy=0 0 0
- added joint right_arm_wrist_pitch_joint: type revolute, parent right_arm_elbow_yaw, child right_arm_wrist_pitch, origin xyz=0.02626 0.018 0.0718 rpy=0 0 0, axis -1 0 0, limit lower=-1.8326 upper=1.8326 effort=100.0 velocity=1.0
- added joint right_arm_wrist_roll_joint: type revolute, parent right_arm_wrist_pitch, child right_arm_wrist_roll, origin xyz=-0.026255 0 0.051425 rpy=0 0 0, axis 0 0 1, limit lower=-2.61799 upper=2.61799 effort=100.0 velocity=1.0
- added joint wheel_left_joint: type continuous, parent base_link, child wheel_left, origin xyz=0.0 0.18 0.095 rpy=1.570796 0 0, axis 0 0 1
- added joint wheel_right_joint: type continuous, parent base_link, child wheel_right, origin xyz=0.0 -0.18 0.095 rpy=1.570796 0 0, axis 0 0 1
- added joint xtion_joint: type fixed, parent bumblebee_link, child xtion_link, origin xyz=0 0 0.055 rpy=0 0 0

Commit message: urdf

File: phoebe.urdf (robot description, URDF)
Before this commit: robot phoebe, 38 links, 37 joints
Joints:
- joint ptu_pan_joint: parent ptu_base_link -> ptu_pan_link
